File: PCB/cc1101.kicad_sch (KiCad schematic)
At the start: 23 parts, among them J5 142-0701-501, U8 CC1101, Y1 26MHz

Commit message: Add files via upload
Parts:
- renumbered J5 to J4, U8 to U6
Changed lines of the file:
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@@
 		(dnp no)
 		(fields_autoplaced yes)
-		(property "Reference" "J5"
+		(property "Reference" "J4"
 			(at 254 110.8709 0)
 			(show_name no)
@@
 			(project "kraky-lite2"
 				(path "/26412b74-f488-4ade-b1b2-7d8b741ec161/39a83b77-a72f-4a92-8517-973f3254d742"
-					(reference "J5")
+					(reference "J4")
 					(unit 1)
 				)
@@
 		(dnp no)
 		(fields_autoplaced yes)
-		(property "Reference" "U8"
+		(property "Reference" "U6"
 			(at 144.2086 128.27 0)
 			(show_name no)
@@
 			(project "kraky-lite2"
 				(path "/26412b74-f488-4ade-b1b2-7d8b741ec161/39a83b77-a72f-4a92-8517-973f3254d742"
-					(reference "U8")
+					(reference "U6")
 					(unit 1)
 				)
