File: PCB/nrf24.kicad_sch (KiCad schematic)
At the start: 18 parts, among them J7 142-0701-501, U5 NRF24L01, Y2 16MHz

Commit message: Add files via upload
Parts:
- renumbered J7 to J6
Changed lines of the file:
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@@
 		(dnp no)
 		(fields_autoplaced yes)
-		(property "Reference" "J7"
+		(property "Reference" "J6"
 			(at 220.98 96.9009 0)
 			(show_name no)
@@
 			(project "kraky-lite2"
 				(path "/26412b74-f488-4ade-b1b2-7d8b741ec161/7beef41a-fa47-464d-bc4f-7a3f1c47524f"
-					(reference "J7")
+					(reference "J6")
 					(unit 1)
 				)
