File: PCB/tfslot.kicad_sch (KiCad schematic)
At the start: 3 parts, among them J6 MSD-4-A

Commit message: Add files via upload
Parts:
- renumbered J6 to J5
Changed lines of the file:
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@@
 		(dnp no)
 		(fields_autoplaced yes)
-		(property "Reference" "J6"
+		(property "Reference" "J5"
 			(at 162.56 100.3299 0)
 			(show_name no)
@@
 			(project "kraky-lite2"
 				(path "/26412b74-f488-4ade-b1b2-7d8b741ec161/c477d776-3a0e-49a9-9044-f493bf435aa9"
-					(reference "J6")
+					(reference "J5")
 					(unit 1)
 				)
