File: PCB/kraky-lite2.kicad_pcb (KiCad board)
At the start: 2 copper layers, 99.2 x 53.9 mm, 83 parts, among them J1 CQ-USB-C16PSMT01, J2 PINHD_1x8_Female, J3 JST_02, J5 142-0701-501, J6 MSD-4-A, J7 142-0701-501, SW1 RotaryEncoder_Switch, SW2 SW_Push, SW3 SW_Push, SW4 SW_Push, SW5 SW_Nidec_CAS-120A1, U1 AMS1117-3.3, U11 ESP32-S3-WROOM-1, U2 AP2112K-3.3TRG1, U3 CH343P, U4 CN3063-SOIC8, U5 NRF24L01, U8 CC1101, Y1 26MHz, Y2 16MHz

Commit message: Add files via upload
Parts:
- added C35: 220 uF, Capacitor_SMD:C_0805_2012Metric, F.Cu at (150.5, 146.8)
- added C36: 220 uF, Capacitor_SMD:C_0805_2012Metric, F.Cu at (145.0, 135.0)
- renumbered J5 to J4, J6 to J5, J7 to J6, U8 to U6, U11 to U7
Routing:
- net GND: track 157.3 -> 165.2 mm
- net Net-(D5-A): track 3.42 -> 6.92 mm
- net 5V: track 77.2 -> 79.9 mm

Commit message: Add files via upload
Parts:
- C35, C36: footprint Capacitor_SMD:C_0805_2012Metric -> Capacitor_SMD:C_1210_3225Metric
- moved C36 4.13 mm to (146.7, 131.2), turned to 180 degrees
- moved C35 0.50 mm to (150.5, 147.2)
Routing:
- net GND: track 165.2 -> 167.2 mm, vias 26 -> 27
- net 5V: track 79.9 -> 81.5 mm
Changed lines of the file:
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@@
 		(tags "Diode SMA (DO-214AC) Handsoldering")
 		(property "Reference" "D5"
-			(at 0 -2.5 0)
+			(at -3.22 -2.425 0)
 			(layer "F.SilkS")
 			(effects
@@
 		)
 	)
-	(footprint "Capacitor_SMD:C_0805_2012Metric"
+	(footprint "Capacitor_SMD:C_1210_3225Metric"
 		(layer "F.Cu")
-		(at 150.5 146.75 180)
-		(descr "Capacitor SMD 0805 (2012 Metric), square (rectangular) end terminal, IPC-7351 nominal, (Body size source: IPC-SM-782 page 76, https://www.pcb-3d.com/wordpress/wp-content/uploads/ipc-sm-782a_amendment_1_and_2.pdf, https://docs.google.com/spreadsheets/d/1BsfQQcO9C6DZCsRaXUlFlo91Tg2WpOkGARC1WS5S8t0/edit?usp=sharing)")
+		(at 150.5 147.25 180)
+		(descr "Capacitor SMD 1210 (3225 Metric), square (rectangular) end terminal, IPC-7351 nominal, (Body size source: IPC-SM-782 page 76, https://www.pcb-3d.com/wordpress/wp-content/uploads/ipc-sm-782a_amendment_1_and_2.pdf)")
 		(tags "capacitor")
 		(property "Reference" "C35"
-			(at 0 -1.68 0)
+			(at 4 -0.5 180)
 			(layer "F.SilkS")
 			(effects
@@
 		)
 		(property "Value" "220 uF"
-			(at 0 1.68 0)
+			(at 0 2.3 180)
 			(layer "F.Fab")
 			(effects
@@
 		)
 		(property "Datasheet" ""
-			(at 0 0 0)
+			(at 0 0 180)
 			(layer "F.Fab")
 			(hide yes)
@@
 		)
 		(property "Description" "Unpolarized capacitor"
-			(at 0 0 0)
+			(at 0 0 180)
 			(layer "F.Fab")
 			(hide yes)
@@
 		)
 		(property "KiLib_Generator" "SMD_2terminal_chip_molded"
-			(at 0 0 0)
+			(at 0 0 180)
 			(layer "F.SilkS")
 			(hide yes)
@@
 		(duplicate_pad_numbers_are_jumpers no)
 		(fp_line
-			(start -0.261252 0.735)
-			(end 0.261252 0.735)
+			(start -0.711252 1.36)
+			(end 0.711252 1.36)
 			(stroke
 				(width 0.12)
@@
 		)
 		(fp_line
-			(start -0.261252 -0.735)
-			(end 0.261252 -0.735)
+			(start -0.711252 -1.36)
+			(end 0.711252 -1.36)
 			(stroke
 				(width 0.12)
@@
 		)
 		(fp_rect
-			(start -1.7 -0.98)
-			(end 1.7 0.98)
+			(start -2.3 -1.6)
+			(end 2.3 1.6)
 			(stroke
 				(width 0.05)
@@
 		)
 		(fp_rect
-			(start -1 -0.625)
-			(end 1 0.625)
+			(start -1.6 -1.25)
+			(end 1.6 1.25)
 			(stroke
 				(width 0.1)
@@
 		)
 		(fp_text user "${REFERENCE}"
-			(at 0 0 0)
+			(at 0 0 180)
 			(layer "F.Fab")
 			(effects
 				(font
-					(size 0.5 0.5)
-					(thickness 0.08)
+					(size 0.8 0.8)
+					(thickness 0.12)
 				)
 			)
 		)
 		(pad "1" smd roundrect
-			(at -0.95 0 180)
-			(size 1 1.45)
+			(at -1.475 0 180)
+			(size 1.15 2.7)
 			(layers "F.Cu" "F.Mask" "F.Paste")
-			(roundrect_rratio 0.25)
+			(roundrect_rratio 0.217391)
 			(net "5V")
 			(pintype "passive")
 		)
 		(pad "2" smd roundrect
-			(at 0.95 0 180)
-			(size 1 1.45)
+			(at 1.475 0 180)
+			(size 1.15 2.7)
 			(layers "F.Cu" "F.Mask" "F.Paste")
-			(roundrect_rratio 0.25)
+			(roundrect_rratio 0.217391)
 			(net "GND")
 			(pintype "passive")
 		)
 		(embedded_fonts no)
-		(model "${KICAD10_3DMODEL_DIR}/Capacitor_SMD.3dshapes/C_0805_2012Metric.step"
+		(model "${KICAD10_3DMODEL_DIR}/Capacitor_SMD.3dshapes/C_1210_3225Metric.step"
 			(offset
 				(xyz 0 0 0)
@@
 		)
 	)
-	(footprint "Capacitor_SMD:C_0805_2012Metric"
+	(footprint "Capacitor_SMD:C_1210_3225Metric"
 		(layer "F.Cu")
-		(at 145 135 90)
-		(descr "Capacitor SMD 0805 (2012 Metric), square (rectangular) end terminal, IPC-7351 nominal, (Body size source: IPC-SM-782 page 76, https://www.pcb-3d.com/wordpress/wp-content/uploads/ipc-sm-782a_amendment_1_and_2.pdf, https://docs.google.com/spreadsheets/d/1BsfQQcO9C6DZCsRaXUlFlo91Tg2WpOkGARC1WS5S8t0/edit?usp=sharing)")
+		(at 146.725 131.25 180)
+		(descr "Capacitor SMD 1210 (3225 Metric), square (rectangular) end terminal, IPC-7351 nominal, (Body size source: IPC-SM-782 page 76, https://www.pcb-3d.com/wordpress/wp-content/uploads/ipc-sm-782a_amendment_1_and_2.pdf)")
 		(tags "capacitor")
 		(property "Reference" "C36"
-			(at 2.5 -0.25 0)
+			(at -4.025 0.25 0)
 			(layer "F.SilkS")
 			(effects
@@
 		)
 		(property "Value" "220 uF"
-			(at 0 1.68 90)
+			(at 0 2.3 0)
 			(layer "F.Fab")
 			(effects
@@
 		)
 		(property "Datasheet" ""
-			(at 0 0 90)
+			(at 0 0 0)
 			(layer "F.Fab")
 			(hide yes)
@@
 		)
 		(property "Description" "Unpolarized capacitor"
-			(at 0 0 90)
+			(at 0 0 0)
 			(layer "F.Fab")
 			(hide yes)
@@
 		)
 		(property "KiLib_Generator" "SMD_2terminal_chip_molded"
-			(at 0 0 90)
+			(at 0 0 0)
 			(layer "F.SilkS")
 			(hide yes)
@@
 		(duplicate_pad_numbers_are_jumpers no)
 		(fp_line
-			(start -0.261252 -0.735)
-			(end 0.261252 -0.735)
+			(start -0.711252 1.36)
+			(end 0.711252 1.36)
 			(stroke
 				(width 0.12)
@@
 		)
 		(fp_line
-			(start -0.261252 0.735)
-			(end 0.261252 0.735)
+			(start -0.711252 -1.36)
+			(end 0.711252 -1.36)
 			(stroke
 				(width 0.12)
@@
 		)
 		(fp_rect
-			(start -1.7 -0.98)
-			(end 1.7 0.98)
+			(start -2.3 -1.6)
+			(end 2.3 1.6)
 			(stroke
 				(width 0.05)
@@
 		)
 		(fp_rect
-			(start -1 -0.625)
-			(end 1 0.625)
+			(start -1.6 -1.25)
+			(end 1.6 1.25)
 			(stroke
 				(width 0.1)
@@
 		)
 		(fp_text user "${REFERENCE}"
-			(at 0 0 90)
+			(at 0 0 0)
 			(layer "F.Fab")
 			(effects
 				(font
-					(size 0.5 0.5)
-					(thickness 0.08)
+					(size 0.8 0.8)
+					(thickness 0.12)
 				)
 			)
 		)
 		(pad "1" smd roundrect
-			(at -0.95 0 90)
-			(size 1 1.45)
+			(at -1.475 0 180)
+			(size 1.15 2.7)
 			(layers "F.Cu" "F.Mask" "F.Paste")
-			(roundrect_rratio 0.25)
+			(roundrect_rratio 0.217391)
 			(net "Net-(D5-A)")
 			(pintype "passive")
 		)
 		(pad "2" smd roundrect
-			(at 0.95 0 90)
-			(size 1 1.45)
+			(at 1.475 0 180)
+			(size 1.15 2.7)
 			(layers "F.Cu" "F.Mask" "F.Paste")
-			(roundrect_rratio 0.25)
+			(roundrect_rratio 0.217391)
 			(net "GND")
 			(pintype "passive")
 		)
 		(embedded_fonts no)
-		(model "${KICAD10_3DMODEL_DIR}/Capacitor_SMD.3dshapes/C_0805_2012Metric.step"
+		(model "${KICAD10_3DMODEL_DIR}/Capacitor_SMD.3dshapes/C_1210_3225Metric.step"
 			(offset
 				(xyz 0 0 0)
@@
 	)
 	(segment
+		(start 141.9 133.6)
+		(end 141.9 135.05)
+		(width 0.2)
+		(layer "F.Cu")
+		(net "GND")
+	)
+	(segment
 		(start 188.5 108.8231)
 		(end 188.0731 109.25)
@@
 	)
 	(segment
+		(start 146.2 144.425)
+		(end 146.2 144.35)
+		(width 0.2)
+		(layer "F.Cu")
+		(net "GND")
+	)
+	(segment
 		(start 113.55 118.25)
 		(end 113.55 119.75)
@@
 	)
 	(segment
-		(start 148.6 146.75)
-		(end 146.2 144.35)
-		(width 0.2)
-		(layer "F.Cu")
-		(net "GND")
-	)
-	(segment
 		(start 127.3 144.6)
 		(end 127.3 147.3)
@@
 	)
 	(segment
-		(start 142.9 134.05)
-		(end 141.9 135.05)
-		(width 0.2)
-		(layer "F.Cu")
-		(net "GND")
-	)
-	(segment
 		(start 115.25 116.55)
 		(end 114.75 117.05)
@@
 	)
 	(segment
-		(start 145 134.05)
-		(end 142.9 134.05)
-		(width 0.2)
-		(layer "F.Cu")
-		(net "GND")
-	)
-	(segment
 		(start 122.8 120.6)
 		(end 122.2 120)
@@
 	)
 	(segment
+		(start 144.5 132)
+		(end 143.5 132)
+		(width 0.2)
+		(layer "F.Cu")
+		(net "GND")
+	)
+	(segment
 		(start 138.625 130.675)
 		(end 139.65 131.7)
@@
 	)
 	(segment
+		(start 145.25 131.25)
+		(end 144.5 132)
+		(width 0.2)
+		(layer "F.Cu")
+		(net "GND")
+	)
+	(segment
 		(start 123.45 125.75)
 		(end 123.45 125.5)
@@
 	)
 	(segment
+		(start 143.5 132)
+		(end 141.9 133.6)
+		(width 0.2)
+		(layer "F.Cu")
+		(net "GND")
+	)
+	(segment
 		(start 157.23 113.73)
 		(end 157.2 113.7)
@@
 	)
 	(segment
-		(start 149.55 146.75)
-		(end 148.6 146.75)
+		(start 149.025 147.25)
+		(end 146.2 144.425)
 		(width 0.2)
 		(layer "F.Cu")
@@
 		(net "GND")
 	)
+	(via
+		(at 143.5 132)
+		(size 0.6)
+		(drill 0.3)
+		(layers "F.Cu" "B.Cu")
+		(free yes)
+		(net "GND")
+	)
 	(segment
 		(start 169.39 137.5)
@@
 	)
 	(segment
-		(start 151.45 146.75)
-		(end 151.45 145)
+		(start 168.25 137.36)
+		(end 168.25 135.55)
 		(width 0.2)
 		(layer "F.Cu")
@@
 	)
 	(segment
-		(start 168.25 137.36)
-		(end 168.25 135.55)
+		(start 185 118.5)
+		(end 185 117.5731)
 		(width 0.2)
 		(layer "F.Cu")
@@
 	)
 	(segment
-		(start 185 118.5)
-		(end 185 117.5731)
+		(start 150.8 146.075)
+		(end 151.975 147.25)
 		(width 0.2)
 		(layer "F.Cu")
@@
 	)
 	(segment
+		(start 150.8 144.35)
+		(end 150.8 146.075)
+		(width 0.2)
+		(layer "F.Cu")
+		(net "5V")
+	)
+	(segment
 		(start 151.45 145)
 		(end 150.8 144.35)
@@
 	)
 	(segment
-		(start 145 135.95)
-		(end 146.905 135.95)
-		(width 0.2)
-		(layer "F.Cu")
-		(net "Net-(D5-A)")
-	)
-	(segment
 		(start 148.5 135.295)
 		(end 148.03 134.825)
@@
 	)
 	(segment
-		(start 146.905 135.95)
-		(end 148.03 134.825)
+		(start 148.03 131.42)
+		(end 148.2 131.25)
+		(width 0.2)
+		(layer "F.Cu")
+		(net "Net-(D5-A)")
+	)
+	(segment
+		(start 148.03 134.825)
+		(end 148.03 131.42)
 		(width 0.2)
 		(layer "F.Cu")
