File: PCB/powersupply.kicad_sch (KiCad schematic)
At the start: 23 parts, among them J1 CQ-USB-C16PSMT01, J3 JST_02, SW5 SW_Nidec_CAS-120A1, U1 AMS1117-3.3, U2 AP2112K-3.3TRG1, U3 CH343P, U4 CN3063-SOIC8

Commit message: Add files via upload
Parts:
- added C35, C36: 220 uF, Capacitor_SMD:C_0805_2012Metric, symbol Device:C
Connections:
- net GND: now also C35.2, C36.2
- net VBUS: now also C35.1
- net at D5.2 (A), U1.2 (VO): now also C36.1
Other:
- moved on the sheet: D5

Commit message: Add files via upload
Parts:
- C35, C36: footprint Capacitor_SMD:C_0805_2012Metric -> Capacitor_SMD:C_1210_3225Metric
Changed lines of the file:
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@@
 			)
 		)
-		(property "Footprint" "Capacitor_SMD:C_0805_2012Metric"
+		(property "Footprint" "Capacitor_SMD:C_1210_3225Metric"
 			(at 134.3152 128.27 0)
 			(hide yes)
@@
 			)
 		)
-		(property "Footprint" "Capacitor_SMD:C_0805_2012Metric"
+		(property "Footprint" "Capacitor_SMD:C_1210_3225Metric"
 			(at 111.4552 128.27 0)
 			(hide yes)
